Commit message: Remove waist roll and pitch joints

File: description/robots/g1/g1_23dof_lock_wrist.urdf (robot description, URDF)
Before this commit: robot g1_29dof_rev_1_0, 39 links, 38 joints
Links:
- removed link waist_roll_link
Joints:
- removed joint waist_pitch_joint
- removed joint waist_roll_joint
- added joint torso_joint: type fixed, parent waist_yaw_link, child torso_link, origin xyz=-0.0039635 0 0.044 rpy=0 0 0
