Commit message: 修改21自由度的配置文件

File: description/robots/g1/g1_21dof_lock_wrist.urdf (robot description, URDF)
Before this commit: robot g1_21dof_rev_1_0, 39 links, 36 joints
Links:
- removed link waist_roll_link
- removed link waist_yaw_link
Joints:
- joint waist_yaw_joint: child waist_yaw_link -> torso_link
